File: 6lp/6lp.sch (KiCad schematic (older format))
At the start: 32 parts, among them J1 MODULE_HEADER, J2 CONN_01X01, J3 CONN_01X04, J4 CONN_02X06, J5 CONN_02X05, J6 USB-MICRO, T1 2450BM15A0015, U1 SAMR21E, X1 CRYSTAL

Commit message: swapped to AT86RF233
Parts:
- removed C9: 100nF, Capacitors_SMD:C_0402, symbol C
- removed D1: TVS-2, SMD_Packages:SOT-23, symbol TVS-2
- removed J2: CONN_01X01, Pin_Headers:Pin_Header_Straight_1x01, symbol CONN_01X01
- removed J3: CONN_01X04, Pin_Headers:Pin_Header_Straight_1x04, symbol CONN_01X04
- removed J4: CONN_02X06, Pin_Headers:Pin_Header_Straight_2x06, symbol CONN_02X06
- removed J5: CONN_02X05, parts:CONN_02x05_0.05in, symbol CONN_02X05
- removed J6: USB-MICRO, parts:MICRO-USB-10104111, symbol USB-MINI-B
- removed U1: SAMR21E, SMD_Packages:QFN-32-1EP, symbol SAMR21E
- added D1, D2, D3, D4: LED, symbol LED
- added R6, R7: 330R, Resistors_SMD:R_0402, symbol R
- added U1: AT86RF233, symbol AT86RF233
- R4, R5: value 10kR -> 330R
- renumbered C11 to C10, C12 to C11, C13 to C12, C14 to C13, C4 to C3, C5 to C4, C3 to C5, C10 to C9
Connections:
- net labels added: D1L, D2L, D3L, D4L, DEVDD, DIG1, DIG2, DIG3, DIG4, EVDD
- net labels removed: +5V, DVDD, EXT_INT, PA06, PA07, PA08, PA09, PA24, PA25, PA27, PA28, SWCLK, SWDIO, VDDANA, VDDCORE
- wire segments 161 -> 125
Other:
- note removed: "IO HEADER"
- note removed: "JTAG"
- note removed: "PROG HEADER"
- moved on the sheet: AE1, C1, C10, C11, C12, C13, C2, C3, C4, C5, C6, C7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

Commit message: at86rf233 sch complete, parts associated
Parts:
- removed X1: CRYSTAL, symbol CRYSTAL
- added R3: 10kR, Resistors_SMD:R_0402, symbol R
- added R4, R5: 0, Resistors_SMD:R_0402, symbol R
- added X1: 16.0000MF09Z-AC3, symbol CRYSTAL-4
- C2: footprint Capacitors_SMD:C_0402 -> Capacitors_SMD:C_0805
- C4: renamed from C3; value C -> 9pF
- C7: renamed from C4; value C -> 9pF; footprint Capacitors_SMD:C_0402 -> Capacitors_SMD:C_0805
- D1, D2, D3, D4: footprint (none) -> LEDs:LED-0603
- U1: footprint (none) -> SMD_Packages:QFN-32-1EP
- renumbered C5 to C3, C6 to C5, C7 to C6, R7 to R10, R3 to R6, R4 to R7, R5 to R8, R6 to R9
Connections:
- net labels added: SLP/~RST, SLP_TR
- net labels removed: ~RESET_OUT
- wire segments 125 -> 166
Other:
- moved on the sheet: C1, C4, C7, D1, D2, D3, D4, J1, R1, R10, R2, R7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

Commit message: text, sch position tweaks
Parts:
- X1: footprint (none) -> parts:TSX-3225
Other:
- note added: "PULL UP FOR ~RESET,\nPULL DOWN FOR SLP_TR"
- moved on the sheet: C10, C2, C3, C4, C5, C6, C7, C8, C9, FB1, X1

Commit message: placement round one...
Parts:
- C7: footprint Capacitors_SMD:C_0805 -> Capacitors_SMD:C_0402
- T1: footprint parts:EIA-0805 -> (none)
Connections:
- net SLP/~RST: now also C1.1, R1.2, R2.2, R3.1, R4.2, R5.2; no longer J1.10 (G3), R1.1
- net CLKM: now reaches R6.1, U1.17 (CLKM)
- new net SLP/~RST~_IO: J1.10 (G3), R1.1
Other:
- moved on the sheet: R6
Changed lines of the file:
@@
 F 0 "C7" H 5250 6200 40  0000 L CNN
 F 1 "9pF" H 5256 6015 40  0000 L CNN
-F 2 "Capacitors_SMD:C_0805" H 5288 5950 30  0001 C CNN
+F 2 "Capacitors_SMD:C_0402" H 5288 5950 30  0001 C CNN
 F 3 "" H 5250 6100 60  0000 C CNN
 	1    5250 6100
@@
 PI_IN
 Text Label 1800 4100 0    60   ~ 0
-SLP/~RST
+SLP/~RST~_IO
 $Comp
 L DGND #PWR013
@@
 Text Label 1800 4000 0    60   ~ 0
 INTERRUPT
-$Comp
-L BALUN-6 T1
-U 1 1 543E821F
-P 8150 3950
-F 0 "T1" H 8500 4200 60  0000 C CNN
-F 1 "2450BM15A0015" H 8150 3950 60  0000 C CNN
-F 2 "parts:EIA-0805" H 8150 3950 60  0001 C CNN
-F 3 "" H 8150 3950 60  0000 C CNN
-	1    8150 3950
-	-1   0    0    -1
-$EndComp
 $Comp
 L AGND #PWR015
@@
 L R R6
 U 1 1 54415717
-P 4250 2900
-F 0 "R6" V 4330 2900 40  0000 C CNN
-F 1 "10kR" V 4257 2901 40  0000 C CNN
-F 2 "Resistors_SMD:R_0402" V 4180 2900 30  0001 C CNN
-F 3 "" H 4250 2900 30  0000 C CNN
-	1    4250 2900
+P 4050 2900
+F 0 "R6" V 4130 2900 40  0000 C CNN
+F 1 "10kR" V 4057 2901 40  0000 C CNN
+F 2 "Resistors_SMD:R_0402" V 3980 2900 30  0001 C CNN
+F 3 "" H 4050 2900 30  0000 C CNN
+	1    4050 2900
 	0    1    1    0
 $EndComp
@@
 L DGND #PWR019
 U 1 1 54415C6A
-P 3900 3000
-F 0 "#PWR019" H 3900 3000 40  0001 C CNN
-F 1 "DGND" H 3900 2930 40  0000 C CNN
-F 2 "" H 3900 3000 60  0000 C CNN
-F 3 "" H 3900 3000 60  0000 C CNN
-	1    3900 3000
+P 3700 3000
+F 0 "#PWR019" H 3700 3000 40  0001 C CNN
+F 1 "DGND" H 3700 2930 40  0000 C CNN
+F 2 "" H 3700 3000 60  0000 C CNN
+F 3 "" H 3700 3000 60  0000 C CNN
+	1    3700 3000
 	1    0    0    -1
 $EndComp
@@
 	5500 1850 5500 2750
 Wire Wire Line
-	4500 2900 4600 2900
+	4300 2900 4600 2900
 Wire Wire Line
 	4600 2900 4600 3050
@@
 	4600 3050 4700 3050
 Wire Wire Line
-	4000 2900 3900 2900
-Wire Wire Line
-	3900 2900 3900 3000
+	3800 2900 3700 2900
+Wire Wire Line
+	3700 2900 3700 3000
 Wire Wire Line
 	3450 4450 3450 4550
@@
 Text Notes 3650 4800 0    60   ~ 0
 PULL UP FOR ~RESET,\nPULL DOWN FOR SLP_TR
+Text Label 3100 4450 0    60   ~ 0
+SLP/~RST
+Text Label 4350 2900 0    60   ~ 0
+CLKM
+$Comp
+L BALUN-6 T1
+U 1 1 543EE96C
+P 8150 3950
+F 0 "T1" H 8500 4200 60  0000 C CNN
+F 1 "2450BM15A0015" H 8150 3950 60  0000 C CNN
+F 2 "" H 8150 3950 60  0000 C CNN
+F 3 "" H 8150 3950 60  0000 C CNN
+	1    8150 3950
+	-1   0    0    -1
+$EndComp
 $EndSCHEMATC

Commit message: closed project for review
Parts:
- added R11, R12: 0, Resistors_SMD:R_0402, symbol R
- T1: footprint (none) -> parts:EIA-0805
Connections:
- net AGND: now also R11.2, R12.2
- net DGND: now also R11.1, R12.1
Changed lines of the file:
@@
 SLP_TR
 Wire Wire Line
-	6000 4550 6000 4650
-Wire Wire Line
-	6000 4650 6000 5050
-Wire Wire Line
-	5300 4650 5400 4650
-Wire Wire Line
-	5400 4650 5500 4650
-Wire Wire Line
-	5500 4650 5600 4650
-Wire Wire Line
-	5600 4650 5700 4650
-Wire Wire Line
-	5700 4650 5800 4650
-Wire Wire Line
-	5800 4650 6000 4650
+	6000 4550 6000 5050
+Wire Wire Line
+	5300 4650 6000 4650
 Wire Wire Line
 	5700 4650 5700 4550
@@
 	6500 4650 6500 4550
 Wire Wire Line
-	6200 4650 6300 4650
-Wire Wire Line
-	6300 4650 6400 4650
-Wire Wire Line
-	6400 4650 6500 4650
-Wire Wire Line
-	6500 4650 6600 4650
-Wire Wire Line
-	6600 4550 6600 4650
-Wire Wire Line
-	6600 4650 6600 5050
+	6200 4650 6600 4650
+Wire Wire Line
+	6600 4550 6600 5050
 Connection ~ 6600 4650
 Wire Wire Line
@@
 	6100 1700 6100 2750
 Wire Wire Line
-	3900 1300 3900 1400
-Wire Wire Line
-	3900 1400 3900 1550
-Wire Wire Line
-	3900 1550 3900 1700
-Wire Wire Line
-	3900 1700 3900 1750
-Wire Wire Line
-	3900 1750 3900 1950
-Wire Wire Line
-	4800 1850 5150 1850
-Wire Wire Line
-	5150 1850 5500 1850
+	3900 1300 3900 1950
+Wire Wire Line
+	4800 1850 5500 1850
 Wire Wire Line
 	5700 1750 5700 2750
@@
 	4800 2350 4800 2500
 Wire Wire Line
-	4800 1400 4800 1850
-Wire Wire Line
-	4800 1850 4800 1950
+	4800 1400 4800 1950
 Connection ~ 4800 1850
 Wire Wire Line
@@
 Connection ~ 3900 1750
 Wire Wire Line
-	3900 1700 4250 1700
-Wire Wire Line
-	4250 1700 5800 1700
+	3900 1700 5800 1700
 Wire Wire Line
 	3550 2500 3550 2350
@@
 	3050 3750 3050 3850
 Wire Wire Line
-	4050 6300 4050 6400
-Wire Wire Line
-	4050 6400 4050 6600
+	4050 6300 4050 6600
 Wire Wire Line
 	4050 6400 5250 6400
@@
 	4600 4250 4700 4250
 Wire Wire Line
-	5250 5350 5250 5800
-Wire Wire Line
-	5250 5800 5250 5900
+	5250 5350 5250 5900
 Wire Wire Line
 	4050 5800 4350 5800
@@
 Connection ~ 4250 1700
 Wire Wire Line
-	10150 3850 10250 3850
-Wire Wire Line
-	10250 3850 10500 3850
+	10150 3850 10500 3850
 Wire Wire Line
 	10250 4000 10250 3850
 Connection ~ 10250 3850
 Wire Wire Line
-	9300 3850 9450 3850
-Wire Wire Line
-	9450 3850 9550 3850
+	9300 3850 9550 3850
 Wire Wire Line
 	9450 4000 9450 3850
@@
 	8850 4050 8850 4500
 Wire Wire Line
-	8850 4500 9450 4500
-Wire Wire Line
-	9450 4500 10250 4500
-Wire Wire Line
-	10250 4400 10250 4500
-Wire Wire Line
-	10250 4500 10250 4650
+	8850 4500 10250 4500
+Wire Wire Line
+	10250 4400 10250 4650
 Wire Wire Line
 	9450 4400 9450 4500
@@
 	8750 4050 8850 4050
 Wire Wire Line
-	8050 4450 8050 4550
-Wire Wire Line
-	8050 4550 8050 4700
+	8050 4450 8050 4700
 Wire Wire Line
 	8050 4550 8250 4550
@@
 Connection ~ 5600 4650
 Wire Wire Line
-	4050 5350 4050 5800
-Wire Wire Line
-	4050 5800 4050 5900
+	4050 5350 4050 5900
 Wire Wire Line
 	2500 4000 2500 3550
@@
 	8300 2900 8650 2900
 Wire Wire Line
-	9250 2000 9250 2300
-Wire Wire Line
-	9250 2300 9250 2600
-Wire Wire Line
-	9250 2600 9250 2900
-Wire Wire Line
-	9250 2900 9250 3000
+	9250 2000 9250 3000
 Wire Wire Line
 	9250 2900 9150 2900
@@
 	4150 4150 4700 4150
 Wire Wire Line
-	2950 4450 3050 4450
-Wire Wire Line
-	3050 4450 3150 4450
-Wire Wire Line
-	3150 4450 3450 4450
-Wire Wire Line
-	3450 4450 3550 4450
-Wire Wire Line
-	3550 4450 3650 4450
+	2950 4450 3650 4450
 Wire Wire Line
 	4150 4450 4600 4450
@@
 F 0 "T1" H 8500 4200 60  0000 C CNN
 F 1 "2450BM15A0015" H 8150 3950 60  0000 C CNN
-F 2 "" H 8150 3950 60  0000 C CNN
+F 2 "parts:EIA-0805" H 8150 3950 60  0001 C CNN
 F 3 "" H 8150 3950 60  0000 C CNN
 	1    8150 3950
 	-1   0    0    -1
 $EndComp
+$Comp
+L AGND #PWR023
+U 1 1 543E1BA0
+P 1950 6350
+F 0 "#PWR023" H 1950 6350 40  0001 C CNN
+F 1 "AGND" H 1950 6280 50  0000 C CNN
+F 2 "" H 1950 6350 60  0000 C CNN
+F 3 "" H 1950 6350 60  0000 C CNN
+	1    1950 6350
+	1    0    0    -1
+$EndComp
+$Comp
+L DGND #PWR024
+U 1 1 543E1BA6
+P 2650 6350
+F 0 "#PWR024" H 2650 6350 40  0001 C CNN
+F 1 "DGND" H 2650 6280 40  0000 C CNN
+F 2 "" H 2650 6350 60  0000 C CNN
+F 3 "" H 2650 6350 60  0000 C CNN
+	1    2650 6350
+	1    0    0    -1
+$EndComp
+$Comp
+L R R11
+U 1 1 543E20DC
+P 2300 6200
+F 0 "R11" V 2380 6200 40  0000 C CNN
+F 1 "0" V 2307 6201 40  0000 C CNN
+F 2 "Resistors_SMD:R_0402" V 2230 6200 30  0001 C CNN
+F 3 "" H 2300 6200 30  0000 C CNN
+	1    2300 6200
+	0    1    1    0
+$EndComp
+Wire Wire Line
+	2550 6200 2650 6200
+Wire Wire Line
+	2650 6000 2650 6350
+Wire Wire Line
+	2050 6200 1950 6200
+Wire Wire Line
+	1950 6000 1950 6350
+$Comp
+L R R12
+U 1 1 543E311A
+P 2300 6000
+F 0 "R12" V 2380 6000 40  0000 C CNN
+F 1 "0" V 2307 6001 40  0000 C CNN
+F 2 "Resistors_SMD:R_0402" V 2230 6000 30  0001 C CNN
+F 3 "" H 2300 6000 30  0000 C CNN
+	1    2300 6000
+	0    1    1    0
+$EndComp
+Wire Wire Line
+	2550 6000 2650 6000
+Wire Wire Line
+	2050 6000 1950 6000
+Connection ~ 2650 6200
+Connection ~ 1950 6200
 $EndSCHEMATC
